File: RevB/S12G-Micro-EVB RevB.brd (EAGLE design)
At the start: 49 x 21 mm, 43 parts, among them IC1 FT232RL, IC2 MCP1640, J2 JUMPER, J3 JUMPER

Commit message: added RevB BOM
Parts:
- R10, R11, R12, R9: value 100 -> 120
Changed lines of the file:
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@@
 <element name="VUSB" library="myLibrary" package="1X1" value="1X1" x="11.54" y="17.81" smashed="yes"/>
 <element name="GND" library="myLibrary" package="1X1" value="1X1" x="37.48" y="17.81" smashed="yes"/>
-<element name="R9" library="myLibrary" package="0805" value="100" x="25.3" y="14.8" smashed="yes" rot="MR270">
+<element name="R9" library="myLibrary" package="0805" value="120" x="25.3" y="14.8" smashed="yes" rot="MR270">
 <attribute name="NAME" x="24.8" y="17.1" size="0.5" layer="26" rot="MR180"/>
 <attribute name="VALUE" x="27.5" y="16.6" size="1.27" layer="28" rot="MR270"/>
 </element>
-<element name="R10" library="myLibrary" package="0805" value="100" x="23.6" y="14.8" smashed="yes" rot="MR90">
+<element name="R10" library="myLibrary" package="0805" value="120" x="23.6" y="14.8" smashed="yes" rot="MR90">
 <attribute name="NAME" x="24.2" y="16.6" size="0.5" layer="26" rot="MR0"/>
 <attribute name="VALUE" x="21.4" y="13" size="1.27" layer="28" rot="MR90"/>
 </element>
-<element name="R11" library="myLibrary" package="0805" value="100" x="20.2" y="14.8" smashed="yes" rot="MR270">
+<element name="R11" library="myLibrary" package="0805" value="120" x="20.2" y="14.8" smashed="yes" rot="MR270">
 <attribute name="NAME" x="19.6" y="17.1" size="0.5" layer="26" rot="MR180"/>
 <attribute name="VALUE" x="22.4" y="16.6" size="1.27" layer="28" rot="MR270"/>
 </element>
-<element name="R12" library="myLibrary" package="0805" value="100" x="21.9" y="14.8" smashed="yes" rot="MR90">
+<element name="R12" library="myLibrary" package="0805" value="120" x="21.9" y="14.8" smashed="yes" rot="MR90">
 <attribute name="NAME" x="22.5" y="16.6" size="0.5" layer="26" rot="MR0"/>
 <attribute name="VALUE" x="19.7" y="13" size="1.27" layer="28" rot="MR90"/>
