File: RevB/S12G-Micro-EVB RevB.sch (EAGLE design)
At the start: 43 parts, among them IC1 FT232RL, IC2 MCP1640, J1 JUMPER_2WAY, J2 JUMPER, J3 JUMPER, J4 JUMPER_2WAY

Commit message: added RevB BOM
Parts:
- R10, R11, R12, R9: value 100 -> 120
Changed lines of the file:
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@@
 <setting verticaltext="up"/>
 </settings>
-<grid distance="0.1" unitdist="inch" unit="inch" style="lines" multiple="1" display="yes" altdistance="0.01" altunitdist="inch" altunit="inch"/>
+<grid distance="0.1" unitdist="inch" unit="inch" style="lines" multiple="1" display="no" altdistance="0.01" altunitdist="inch" altunit="inch"/>
 <layers>
 <layer number="1" name="Top" color="4" fill="1" visible="no" active="no"/>
@@
 <part name="VUSB" library="myLibrary" deviceset="1X1" device=""/>
 <part name="GND" library="myLibrary" deviceset="1X1" device=""/>
-<part name="R9" library="myLibrary" deviceset="R" device="" value="100"/>
-<part name="R10" library="myLibrary" deviceset="R" device="" value="100"/>
-<part name="R11" library="myLibrary" deviceset="R" device="" value="100"/>
-<part name="R12" library="myLibrary" deviceset="R" device="" value="100"/>
+<part name="R9" library="myLibrary" deviceset="R" device="" value="120"/>
+<part name="R10" library="myLibrary" deviceset="R" device="" value="120"/>
+<part name="R11" library="myLibrary" deviceset="R" device="" value="120"/>
+<part name="R12" library="myLibrary" deviceset="R" device="" value="120"/>
 <part name="R13" library="myLibrary" deviceset="R" device="" value="10K"/>
 <part name="GND6" library="supply1" deviceset="GND" device=""/>
